File: HW2/ME433/ME433.sch (EAGLE design)
At the start: 22 parts, among them J1 USB-MB-H

Commit message: eagle schematic
Parts:
- C1, C2, C3, C4: value (none) -> 0.1
- C5, C6: value (none) -> 10
- LED1: value (none) -> Red
- LED2: value (none) -> Green
- R1, R2: value (none) -> 330
- R3, R4: value (none) -> 10k
- U$4: value PB -> RESET
- U$5: value PB -> USER
- U$7: value OSC -> 8MHz
Connections:
- new net +3V3: C1.1, C2.1, C4.1, C6.+, J3.2, LED1.A, R3.2, R4.2, U$1.13.VDD, U$1.23.VUSB3V3, U$1.28.AVDD, U$3.3.VOUT, U$6.VDD
- new net +5V: C3.1, J2.2, U$1.15.VBUS, U$2.1, U$3.2.VIN
- new net A0: J3.8, U$1.2.A0
- new net A1: J3.7, U$1.3.A1
- new net A4/LED: J3.3, LED2.A, U$1.12.A4/LED
- new net B13: J2.6, U$1.24.B13
- new net B14: J2.7, U$1.25.B14
- new net B15: J2.8, U$1.26.B15
- new net B2: J3.6, U$1.6.B2
- new net B3: J3.5, U$1.7.B3
- new net B4/USER: J3.4, R4.1, U$1.11.B4/USER, U$5.1
- new net B7: J2.3, U$1.16.B7
- new net B8: J2.4, U$1.17.B8
- new net B9: J2.5, U$1.18.B9
- new net D+: J1.D+, U$1.21.D+/BI0
- new net D-: J1.D-, U$1.22.D-/B11
- new net GND: C1.2, C2.2, C3.2, C4.2, C5.-, C6.-, J1.GND, J2.1, J3.1, R1.1, R2.1, U$1.17.AVSS, U$1.19.VSS, U$1.8.VSS, U$3.1.GND, U$4.2, U$5.2, U$6.GND, U$7.2.GND
- new net MCLR: R3.1, U$1.1.MCLR, U$4.1, U$6.MCLR
- new net N$1: J1.VBUS, U$2.2
- new net N$2: LED2.C, R2.2
- new net N$3: LED1.C, R1.2
- new net N$4: U$1.9.OSC1/A2, U$7.1.OSC1
- new net N$5: U$1.10.OSC2/A3, U$7.3.OSC2
- new net N$7: C5.+, U$1.20.VCAP
- new net PGC: U$1.5.PGC/B1, U$6.PGC
- new net PGD: U$1.4.PGD/B0, U$6.PGD
- new net USBID: J1.ID, U$1.14.USBID/B5
Other:
- moved on the sheet: C1, C2, C3, C4, C5, C6, J2, J3, LED1, LED2, R1, R2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
